File: ACCIO/Closed Loop Motor Control PCB/ClosedLoopMotorControlPCB/ClosedLoopMotorControlPCB.kicad_pcb (KiCad board)
At the start: 2 copper layers, 83.8 x 66 mm, 50 parts, among them J1 Conn_01x03, J2 +24V_IN, J3 MD13S_control, J4 MD13S_power, J5 MD13S_toMotor, J6 Motor, J7 Conn_01x04, J8 LIMIT_SWITCH1, J9 LIMIT_SWITCH2, Q1 AO3401A, SW1 RST Button, SW2 BOOT Button, U1 ESP32-WROOM-32E, U2 LM2596S-5, U3 AMS1117-3.3, U4 INA219AxD

Commit message: accio task update
Routing:
- net GND: track 1.41 -> 66.0 mm, vias 0 -> 1
- net Net-(U1-IO0): track 31.2 -> 40.8 mm
- net +24V_RAIL: track 161.2 -> 162.5 mm
Changed lines of the file:
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@@
 		(tags "resistor")
 		(property "Reference" "R2"
-			(at 0.9125 5.08 0)
+			(at 0.9125 0 0)
 			(layer "F.SilkS")
+			(hide yes)
 			(effects
 				(font
@@
 		(net 1)
 	)
+	(via
+		(at 194.31 80.65)
+		(size 0.6)
+		(drill 0.3)
+		(layers "F.Cu" "B.Cu")
+		(free yes)
+		(net 1)
+	)
+	(segment
+		(start 187.96 76.01)
+		(end 197.93 76.01)
+		(width 0.2)
+		(layer "B.Cu")
+		(net 1)
+	)
+	(segment
+		(start 167.64 81.507677)
+		(end 167.64 86.36)
+		(width 0.2)
+		(layer "B.Cu")
+		(net 1)
+	)
+	(segment
+		(start 197.93 76.01)
+		(end 205.74 83.82)
+		(width 0.2)
+		(layer "B.Cu")
+		(net 1)
+	)
+	(segment
+		(start 164.925 78.792677)
+		(end 167.64 81.507677)
+		(width 0.2)
+		(layer "B.Cu")
+		(net 1)
+	)
+	(segment
+		(start 175.8925 94.6125)
+		(end 175.8925 96.255)
+		(width 0.2)
+		(layer "B.Cu")
+		(net 1)
+	)
+	(segment
+		(start 167.64 86.36)
+		(end 175.8925 94.6125)
+		(width 0.2)
+		(layer "B.Cu")
+		(net 1)
+	)
+	(segment
+		(start 202.070062 80.150062)
+		(end 205.74 83.82)
+		(width 0.2)
+		(layer "B.Cu")
+		(net 1)
+	)
+	(segment
+		(start 194.31 80.65)
+		(end 194.809938 80.150062)
+		(width 0.2)
+		(layer "B.Cu")
+		(net 1)
+	)
+	(segment
+		(start 194.809938 80.150062)
+		(end 202.070062 80.150062)
+		(width 0.2)
+		(layer "B.Cu")
+		(net 1)
+	)
+	(segment
+		(start 200.66 88.9)
+		(end 205.74 83.82)
+		(width 0.2)
+		(layer "B.Cu")
+		(net 1)
+	)
+	(segment
+		(start 199.39 88.9)
+		(end 200.66 88.9)
+		(width 0.2)
+		(layer "B.Cu")
+		(net 1)
+	)
 	(segment
 		(start 210.072 55.88)
@@
 	)
 	(segment
+		(start 198.12 97.22)
+		(end 198.12 95.95)
+		(width 0.2)
+		(layer "F.Cu")
+		(net 4)
+	)
+	(segment
 		(start 169.555 68.255)
 		(end 171.625 66.185)
@@
 	)
 	(segment
-		(start 193.4375 77.43)
-		(end 183.5065 87.361)
+		(start 181.055 89.615)
+		(end 182.88 91.44)
 		(width 0.2)
 		(layer "F.Cu")
@@
 	)
 	(segment
-		(start 183.5065 87.361)
-		(end 182.056 87.361)
+		(start 186.758 91.44)
+		(end 182.88 91.44)
 		(width 0.2)
 		(layer "F.Cu")
@@
 	)
 	(segment
-		(start 182.056 87.361)
-		(end 181.055 86.36)
+		(start 181.055 86.36)
+		(end 180.050064 86.36)
+		(width 0.2)
+		(layer "F.Cu")
+		(net 24)
+	)
+	(segment
+		(start 193.4375 77.43)
+		(end 187.359 83.5085)
+		(width 0.2)
+		(layer "F.Cu")
+		(net 24)
+	)
+	(segment
+		(start 187.359 83.5085)
+		(end 187.359 90.839)
 		(width 0.2)
 		(layer "F.Cu")
@@
 	(segment
 		(start 181.055 86.36)
-		(end 180.050064 86.36)
+		(end 181.055 89.615)
 		(width 0.2)
 		(layer "F.Cu")
@@
 		(width 0.2)
 		(layer "F.Cu")
+		(net 24)
+	)
+	(segment
+		(start 187.359 90.839)
+		(end 186.758 91.44)
+		(width 0.2)
+		(layer "F.Cu")
